File: HACKberry-hardware/electronics/SensorBoard_v1/SensorBoard_v1.sch (KiCad schematic (older format))
At the start: 0 parts

Commit message: bug fix
Parts:
- added R1: 300, symbol R
- added R2: 10k, symbol R
- added U1: 3-CONDUCTOR_MINIATUIRE_JACK_MJ-4535-3, symbol 3-CONDUCTOR_MINIATUIRE_JACK_MJ-4535-3
- added U2: TPR-105, symbol TPR-105
Connections:
- new net: R1.2, U1.1 (INPUT), U2.4 (Emitter)
- new net: U1.2 (VCC), U2.1 (Anode), U2.3 (Collector)
- new net: R1.1, R2.1, U1.3 (GND)
- new net: R2.2, U2.2 (Cathode)
Changed lines of the file:
@@
 LIBS:contrib
 LIBS:valves
+LIBS:yamaura
+LIBS:SensorBoard_v1-cache
 EELAYER 25 0
 EELAYER END
@@
 encoding utf-8
 Sheet 1 1
-Title ""
+Title "SensorBoard_v1"
 Date ""
 Rev ""
-Comp ""
+Comp "exiii"
 Comment1 ""
 Comment2 ""
@@
 Comment4 ""
 $EndDescr
+$Comp
+L 3-CONDUCTOR_MINIATUIRE_JACK_MJ-4535-3 U1
+U 1 1 55601F64
+P 4750 4000
+F 0 "U1" H 4550 4300 60  0000 C CNN
+F 1 "3-CONDUCTOR_MINIATUIRE_JACK_MJ-4535-3" H 4750 4200 60  0000 C CNN
+F 2 "" H 4750 4200 60  0000 C CNN
+F 3 "" H 4750 4200 60  0000 C CNN
+	1    4750 4000
+	1    0    0    -1
+$EndComp
+$Comp
+L TPR-105 U2
+U 1 1 55602C89
+P 6550 3950
+F 0 "U2" H 6550 4150 60  0000 C CNN
+F 1 "TPR-105" H 6550 3750 60  0000 C CNN
+F 2 "" H 6550 3950 60  0000 C CNN
+F 3 "" H 6550 3950 60  0000 C CNN
+	1    6550 3950
+	-1   0    0    1
+$EndComp
+$Comp
+L R R1
+U 1 1 55602FD5
+P 6950 3350
+F 0 "R1" V 7030 3350 50  0000 C CNN
+F 1 "300" V 6950 3350 50  0000 C CNN
+F 2 "" V 6880 3350 30  0000 C CNN
+F 3 "" H 6950 3350 30  0000 C CNN
+	1    6950 3350
+	0    1    1    0
+$EndComp
+$Comp
+L R R2
+U 1 1 55603071
+P 6950 4500
+F 0 "R2" V 7030 4500 50  0000 C CNN
+F 1 "10k" V 6950 4500 50  0000 C CNN
+F 2 "" V 6880 4500 30  0000 C CNN
+F 3 "" H 6950 4500 30  0000 C CNN
+	1    6950 4500
+	0    1    1    0
+$EndComp
+Wire Wire Line
+	5100 3900 6000 3900
+Wire Wire Line
+	6800 3350 6000 3350
+Wire Wire Line
+	6000 3350 6000 3900
+Wire Wire Line
+	5100 4000 6000 4000
+Wire Wire Line
+	7100 4000 7100 4200
+Wire Wire Line
+	7100 4200 6800 4200
+Wire Wire Line
+	6800 4200 6800 4500
+Wire Wire Line
+	7100 3350 7200 3350
+Wire Wire Line
+	7200 4500 7100 4500
+Wire Wire Line
+	7100 3900 7150 3900
+Wire Wire Line
+	7150 4300 6000 4300
+Wire Wire Line
+	6000 4300 6000 4000
+Wire Wire Line
+	5100 4100 5950 4100
+Wire Wire Line
+	5950 4100 5950 4650
+Wire Wire Line
+	5950 4650 7200 4650
+Connection ~ 7200 4500
+Connection ~ 7150 3900
+Connection ~ 7200 4650
+Wire Wire Line
+	7200 4650 7200 3350
+Wire Wire Line
+	7150 3900 7150 4300
 $EndSCHEMATC
