File: HACKberry-hardware/electronics/SensorBoard_v1/SensorBoard_v1.kicad_pcb (KiCad board)
At the start: 2 copper layers, 27.9 x 25.4 mm, 6 parts, among them U1 3-CONDUCTOR_MINIATUIRE_JACK_M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, U2 TPR-105

Commit message: Fixed minor error
Parts:
- REF** (x2): value SolderWirePad_single_2mmDrill -> (none)
- moved U1 128.3 mm to (120.3, 104.7)
- moved REF** 128.2 mm to (126.5, 114.9)
- moved U2 128.2 mm to (132.7, 104.8)
- moved R1 128.2 mm to (132.7, 100.7)
- moved R2 128.2 mm to (132.7, 108.7)
- moved REF** 128.2 mm to (139.1, 94.5)
