File: HACKberry-hardware/electronics/HandBoard_v1/HandBoard_v1.sch (KiCad schematic (older format))
At the start: 11 parts, among them CON1 BARREL_JACK_MJ179PH, SW1 SW_PUSH_SKRGAQD010, SW2 SW_PUSH_SKRGAQD010, SW3 SW_PUSH_SKRGAQD010, SW4 SWITCH_SS-12SDP2, U2 3-CONDUCTOR_MINIATUIRE_JACK_M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, U3 Arduino_Micro, U4 Seed_Studio_Adjustable_DC/DC_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, U5 Servo_Motor_MG90S, U6 Servo_Motor_S03N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

Commit message: Modified the schematic.
Added the push switch.
Parts:
- added SW4: SW_PUSH, symbol SW_PUSH
- CON1: footprint (none) -> HACKberry_v1:MJ179PH
- SW1, SW2, SW3: footprint (none) -> HACKberry_v1:SKRGAQ0010
- SW5: renamed from SW4; footprint (none) -> Pin_Headers:Pin_Header_Straight_1x03
- U1: renamed from U2; footprint (none) -> HACKberry_v1:MINIATURE_JACK_MJ-4535-3
- U2: renamed from U3; footprint (none) -> HACKberry_v1:Arduino_Micro
- U4: renamed from U5; footprint (none) -> Pin_Headers:Pin_Header_Straight_1x03
- U5: renamed from U6; footprint (none) -> Pin_Headers:Pin_Header_Straight_1x03
- U6: renamed from U7; footprint (none) -> Pin_Headers:Pin_Header_Straight_1x03
- renumbered U4 to U3
Connections:
- wire segments 57 -> 59
- no-connect marks 22 -> 21
Changed lines of the file:
@@
 EESchema Schematic File Version 2
+LIBS:myParts
 LIBS:power
 LIBS:device
@@
 $EndDescr
 $Comp
-L Arduino_Micro U3
+L Arduino_Micro U2
 U 1 1 555EFCA5
 P 5500 4000
-F 0 "U3" H 5500 5000 60  0000 C CNN
+F 0 "U2" H 5500 5000 60  0000 C CNN
 F 1 "Arduino_Micro" H 5500 3050 60  0000 C CNN
-F 2 "" V 5500 4000 60  0000 C CNN
+F 2 "HACKberry_v1:Arduino_Micro" V 5500 4000 60  0001 C CNN
 F 3 "" V 5500 4000 60  0000 C CNN
 	1    5500 4000
@@
 $EndComp
 $Comp
-L Servo_Motor U5
+L Servo_Motor U4
 U 1 1 555F1F15
 P 8000 3650
-F 0 "U5" H 7800 3950 60  0000 C CNN
+F 0 "U4" H 7800 3950 60  0000 C CNN
 F 1 "Servo_Motor_MG90S" H 8000 3850 60  0000 C CNN
-F 2 "" H 8000 3850 60  0000 C CNN
+F 2 "Pin_Headers:Pin_Header_Straight_1x03" H 8000 3850 60  0001 C CNN
 F 3 "" H 8000 3850 60  0000 C CNN
 	1    8000 3650
@@
 $EndComp
 $Comp
-L Servo_Motor U6
+L Servo_Motor U5
 U 1 1 555F20CE
 P 8000 4150
-F 0 "U6" H 7800 4450 60  0000 C CNN
+F 0 "U5" H 7800 4450 60  0000 C CNN
 F 1 "Servo_Motor_S03N" H 8000 4350 60  0000 C CNN
-F 2 "" H 8000 4350 60  0000 C CNN
+F 2 "Pin_Headers:Pin_Header_Straight_1x03" H 8000 4350 60  0001 C CNN
 F 3 "" H 8000 4350 60  0000 C CNN
 	1    8000 4150
@@
 $EndComp
 $Comp
-L Servo_Motor U7
+L Servo_Motor U6
 U 1 1 555F20F9
 P 8000 4650
-F 0 "U7" H 7800 4950 60  0000 C CNN
+F 0 "U6" H 7800 4950 60  0000 C CNN
 F 1 "Servo_Motor_MG90S" H 8000 4850 60  0000 C CNN
-F 2 "" H 8000 4850 60  0000 C CNN
+F 2 "Pin_Headers:Pin_Header_Straight_1x03" H 8000 4850 60  0001 C CNN
 F 3 "" H 8000 4850 60  0000 C CNN
 	1    8000 4650
@@
 $EndComp
 $Comp
-L Seed_Studio_Adjustable_DC/DC_Power_Converter_(1.25V_-_35V/3A) U4
+L Seed_Studio_Adjustable_DC/DC_Power_Converter_(1.25V_-_35V/3A) U3
 U 1 1 555F2DA3
 P 5500 5400
-F 0 "U4" H 5500 5650 60  0000 C CNN
+F 0 "U3" H 5500 5650 60  0000 C CNN
 F 1 "Seed_Studio_Adjustable_DC/DC_Power_Converter_(1.25V_-_35V/3A)" H 5550 5150 60  0000 C CNN
-F 2 "" H 5550 5150 60  0000 C CNN
+F 2 "" H 5550 5150 60  0001 C CNN
 F 3 "" H 5550 5150 60  0000 C CNN
 	1    5500 5400
@@
 $EndComp
 $Comp
-L 3-CONDUCTOR_MINIATUIRE_JACK_MJ-4535-3 U2
+L 3-CONDUCTOR_MINIATUIRE_JACK_MJ-4535-3 U1
 U 1 1 555F3180
-P 3200 4500
-F 0 "U2" H 3000 4800 60  0000 C CNN
-F 1 "3-CONDUCTOR_MINIATUIRE_JACK_MJ-4535-3" H 3200 4700 60  0000 C CNN
-F 2 "" H 3200 4700 60  0000 C CNN
-F 3 "" H 3200 4700 60  0000 C CNN
-	1    3200 4500
+P 3200 4700
+F 0 "U1" H 3000 5000 60  0000 C CNN
+F 1 "3-CONDUCTOR_MINIATUIRE_JACK_MJ-4535-3" H 3200 4900 60  0000 C CNN
+F 2 "HACKberry_v1:MINIATURE_JACK_MJ-4535-3" H 3200 4900 60  0001 C CNN
+F 3 "" H 3200 4900 60  0000 C CNN
+	1    3200 4700
 	1    0    0    -1
 $EndComp
@@
 F 0 "SW1" H 3350 3310 50  0000 C CNN
 F 1 "SW_PUSH_SKRGAQD010" H 3200 3120 50  0000 C CNN
-F 2 "" H 3200 3200 60  0000 C CNN
+F 2 "HACKberry_v1:SKRGAQ0010" H 3200 3200 60  0001 C CNN
 F 3 "" H 3200 3200 60  0000 C CNN
 	1    3200 3200
@@
 F 0 "SW2" H 3350 3610 50  0000 C CNN
 F 1 "SW_PUSH_SKRGAQD010" H 3200 3420 50  0000 C CNN
-F 2 "" H 3200 3500 60  0000 C CNN
+F 2 "HACKberry_v1:SKRGAQ0010" H 3200 3500 60  0001 C CNN
 F 3 "" H 3200 3500 60  0000 C CNN
 	1    3200 3500
@@
 F 0 "SW3" H 3350 3910 50  0000 C CNN
 F 1 "SW_PUSH_SKRGAQD010" H 3200 3720 50  0000 C CNN
-F 2 "" H 3200 3800 60  0000 C CNN
+F 2 "HACKberry_v1:SKRGAQ0010" H 3200 3800 60  0001 C CNN
 F 3 "" H 3200 3800 60  0000 C CNN
 	1    3200 3800
@@
 $EndComp
 $Comp
-L SWITCH_INV SW4
+L SWITCH_INV SW5
 U 1 1 555F35ED
 P 4300 5200
-F 0 "SW4" H 4100 5350 50  0000 C CNN
+F 0 "SW5" H 4100 5350 50  0000 C CNN
 F 1 "SWITCH_SS-12SDP2" H 4250 5000 50  0000 C CNN
-F 2 "" H 4300 5200 60  0000 C CNN
+F 2 "Pin_Headers:Pin_Header_Straight_1x03" H 4300 5200 60  0001 C CNN
 F 3 "" H 4300 5200 60  0000 C CNN
 	1    4300 5200
@@
 NoConn ~ 4750 4400
 NoConn ~ 4750 4300
-NoConn ~ 4750 4200
 NoConn ~ 4750 3700
 NoConn ~ 4750 3600
@@
 	4350 3500 4350 5000
 Wire Wire Line
-	4350 4600 3550 4600
+	4350 4800 3550 4800
 Wire Wire Line
 	4350 5000 3850 5000
 Connection ~ 3850 5300
-Connection ~ 4350 4600
+Connection ~ 4350 4800
 Wire Wire Line
 	2900 3200 2650 3200
 Wire Wire Line
-	2650 3200 2650 4150
+	2650 3200 2650 4300
 Wire Wire Line
 	2650 3500 2900 3500
@@
 Connection ~ 2650 3500
 Wire Wire Line
-	2650 4150 4350 4150
-Connection ~ 4350 4150
+	2650 4300 4350 4300
+Connection ~ 4350 4300
 Connection ~ 2650 3800
 Wire Wire Line
@@
 F 0 "CON1" H 3050 5450 60  0000 C CNN
 F 1 "BARREL_JACK_MJ179PH" H 3050 5000 60  0000 C CNN
-F 2 "" H 3050 5200 60  0000 C CNN
+F 2 "HACKberry_v1:MJ179PH" H 3050 5200 60  0001 C CNN
 F 3 "" H 3050 5200 60  0000 C CNN
 	1    3050 5200
@@
 NoConn ~ 3350 5200
 Wire Wire Line
-	3550 4500 4450 4500
-Wire Wire Line
-	4450 4500 4450 4700
-Wire Wire Line
-	4450 4700 4750 4700
-Wire Wire Line
-	3550 4400 4550 4400
-Wire Wire Line
-	4550 4400 4550 4500
+	3550 4700 4750 4700
+Wire Wire Line
+	3550 4600 4550 4600
+Wire Wire Line
+	4550 4600 4550 4500
 Wire Wire Line
 	4550 4500 4750 4500
 Connection ~ 4900 5100
+$Comp
+L SW_PUSH SW4
+U 1 1 5573938F
+P 3200 4050
+F 0 "SW4" H 3350 4160 50  0000 C CNN
+F 1 "SW_PUSH" H 3200 3970 50  0000 C CNN
+F 2 "" H 3200 4050 60  0000 C CNN
+F 3 "" H 3200 4050 60  0000 C CNN
+	1    3200 4050
+	1    0    0    -1
+$EndComp
+Wire Wire Line
+	2900 4050 2650 4050
+Connection ~ 2650 4050
+Wire Wire Line
+	3500 4050 3700 4050
+Wire Wire Line
+	3700 4050 3700 4200
+Wire Wire Line
+	3700 4200 4750 4200
 $EndSCHEMATC
