File: HACKberry-hardware/electronics/HandBoard_v1/HandBoard_v1.kicad_pcb (KiCad board)
At the start: 2 copper layers, 60.8 x 54.8 mm, 10 parts, among them CON1 BARREL_JACK_MJ179PH, SW1 SW_PUSH_SKRGAQD010, SW2 SW_PUSH_SKRGAQD010, SW3 SW_PUSH_SKRGAQD010, SW4 SWITCH_SS-12SDP2, U2 3-CONDUCTOR_MINIATUIRE_JACK_M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, U3 Arduino_Micro, U5 Servo_Motor_MG90S, U6 Servo_Motor_S03N, U7 Servo_Motor_MG90S

Commit message: Proceeded detail design of the hand boad
Parts:
- added SW1: SW_PUSH_SKRGAQD010, HACKberry_v1:SKRGAQ0010, F.Cu at (54.9, 92.6)
- SW4: value SWITCH_SS-12SDP2 -> SW_PUSH
- U2: value 3-CONDUCTOR_MINIATUIRE_JACK_MJ-4535-3 -> Arduino_Micro
- U3: value Arduino_Micro -> Seed_Studio_Adjustable_DC/DC_Power_Converter_(1.25V_-_35V/3A)
- U5: value Servo_Motor_MG90S -> Servo_Motor_S03N
- U6: value Servo_Motor_S03N -> Servo_Motor_MG90S
Connections:
- SW4 pad 1: Net-(SW4-Pad1) -> Net-(CON1-Pad3)
- SW4 pad 2: Net-(CON1-Pad1) -> Net-(SW4-Pad2)
- SW4 pad 3: Net-(SW4-Pad3) -> (no net)
- U2 pad 1: Net-(CON1-Pad3) -> (no net)
- U2 pad 4: Net-(U2-Pad4) -> (no net)
- U3 pad 10: Net-(U3-Pad10) -> (no net)
- U3 pad 11: Net-(U3-Pad11) -> (no net)
- U3 pad 12: Net-(U3-Pad12) -> (no net)
- U3 pad 13: Net-(U3-Pad13) -> (no net)
- U3 pad 2: Net-(U3-Pad2) -> Net-(CON1-Pad3)
- U3 pad 5: Net-(U3-Pad5) -> (no net)
- U3 pad 5V: Net-(U3-Pad5V) -> (no net)
- U3 pad 6: Net-(U3-Pad6) -> (no net)
- U3 pad 7: Net-(U3-Pad7) -> (no net)
- U3 pad 8: Net-(U3-Pad8) -> (no net)
- U3 pad A0: Net-(U2-Pad2) -> (no net)
- U3 pad A1: Net-(U3-PadA1) -> (no net)
- U3 pad A2: Net-(U3-PadA2) -> (no net)
- U3 pad A3: Net-(U3-PadA3) -> (no net)
- U3 pad A4: Net-(SW3-Pad2) -> (no net)
- U3 pad A5: Net-(SW2-Pad2) -> (no net)
- U3 pad A6: Net-(SW1-Pad2) -> (no net)
- U3 pad GND: Net-(U3-PadGND) -> (no net)
- U3 pad MISO: Net-(U3-PadMISO) -> (no net)
- U3 pad NC: Net-(U3-PadNC) -> (no net)
- U3 pad RESE: Net-(U3-PadRESE) -> (no net)
- U3 pad RST: Net-(U3-PadRST) -> (no net)
- U3 pad RX: Net-(U3-PadRX) -> (no net)
- U3 pad SCK: Net-(U3-PadSCK) -> (no net)
- U3 pad SS: Net-(U3-PadSS) -> (no net)
- U3 pad TX: Net-(U3-PadTX) -> (no net)
- U3 pad VIN: Net-(SW4-Pad1) -> (no net)
- U5 pad 1: Net-(U3-Pad3) -> Net-(U2-Pad5)
- U5 pad 2: Net-(U4-Pad4) -> Net-(U3-Pad4)
- U5 pad 3: Net-(U4-Pad3) -> Net-(U3-Pad3)
- U6 pad 1: Net-(U3-Pad5) -> Net-(U2-Pad6)
- U6 pad 2: Net-(U4-Pad4) -> Net-(U3-Pad4)
- U6 pad 3: Net-(U4-Pad3) -> Net-(U3-Pad3)
Routing:
- net (no net): track 0.00 -> 40.9 mm
- net Net-(U2-Pad2): track 0.00 -> 8.31 mm
Other:
- outline, holes or cut-outs redrawn
- net class Default: trace_width 0.25 -> 0.5
